File: boards/adsb-test/hardware/kicad/m1421.kicad_sch (KiCad schematic)
At the start: 0 parts

Commit message: Release v0.15.0: KiCad sheet generator, ADSB_Test M1421 schematic with Dev Kit header
Co-Authored-By: Claude Opus 5.5 <noreply@anthropic.com>
Parts:
- added C1401: 1uF, Capacitor_SMD:C_0402_1005Metric, symbol Device:C
- added C1402: 100nF, Capacitor_SMD:C_0402_1005Metric, symbol Device:C
- added D1401: RED 1090, LED_SMD:LED_0603_1608Metric, symbol Device:LED
- added D1402: GREEN UAT, LED_SMD:LED_0603_1608Metric, symbol Device:LED
- added D1403: ESD7351XV2T1G, Diode_SMD:D_SOD-523, symbol Device:D_TVS
- added J1401: m1421 JTAG (J-Link), Connector_PinHeader_1.27mm:PinHeader_2x05_P1.27mm_Vertical_SMD, symbol Connector:Conn_ARM_JTAG_SWD_10
- added J1402: ADSBee 1421 Dev Kit, Connector_PinHeader_2.54mm:PinHeader_1x06_P2.54mm_Vertical, symbol Connector_Generic:Conn_01x06
- added J1403: SMA 1090/978, Connector_Coaxial:SMA_Samtec_SMA-J-P-H-ST-EM1_EdgeMount, symbol Connector:Conn_Coaxial
- added R1401, R1402, R1403, R1404, R1405: 100k, Resistor_SMD:R_0402_1005Metric, symbol Device:R
- added R1406: 287R, Resistor_SMD:R_0402_1005Metric, symbol Device:R
- added R1407: 115R, Resistor_SMD:R_0402_1005Metric, symbol Device:R
- added R1408: 100R, Resistor_SMD:R_0402_1005Metric, symbol Device:R
- added TP1401: SD23, TestPoint:TestPoint_Pad_D1.0mm, symbol Connector:TestPoint
- added TP1402: SD24, TestPoint:TestPoint_Pad_D1.0mm, symbol Connector:TestPoint
- added TP1403: SD25, TestPoint:TestPoint_Pad_D1.0mm, symbol Connector:TestPoint
- added TP1404: LD11, TestPoint:TestPoint_Pad_D1.0mm, symbol Connector:TestPoint
- added TP1405: LD09, TestPoint:TestPoint_Pad_D1.0mm, symbol Connector:TestPoint
- added TP1406: LD08, TestPoint:TestPoint_Pad_D1.0mm, symbol Connector:TestPoint
- added TP1407: LRST, TestPoint:TestPoint_Pad_D1.0mm, symbol Connector:TestPoint
- added TP1408: CSMI, TestPoint:TestPoint_Pad_D1.0mm, symbol Connector:TestPoint
- added TP1409: CSMO, TestPoint:TestPoint_Pad_D1.0mm, symbol Connector:TestPoint
- added TP1410: CSCK, TestPoint:TestPoint_Pad_D1.0mm, symbol Connector:TestPoint
- added TP1411: LRCS, TestPoint:TestPoint_Pad_D1.0mm, symbol Connector:TestPoint
- added TP1412: LBSY, TestPoint:TestPoint_Pad_D1.0mm, symbol Connector:TestPoint
- added U1401: ADSBee m1421, ADSB_Test:PantsForBirds_ADSBee_m1421_Module, symbol ADSB_Test:PantsForBirds_ADSBee_m1421
- added U1402: 74LVC1G97 (2:1 mux), Package_TO_SOT_SMD:SOT-363_SC-70-6, symbol 74xGxx:74LVC1G97
- added U1403: 74LVC1G32, Package_TO_SOT_SMD:SOT-353_SC-70-5, symbol 74xGxx:74LVC1G32
- added U1404: 74LVC1G07, Package_TO_SOT_SMD:SOT-353_SC-70-5, symbol 74xGxx:74LVC1G07
- added U1405: SCN-2-11+, ADSB_Test:MiniCircuits_SCN, symbol ADSB_Test:MiniCircuits_SCN-2-11
Connections:
- new net 3V3_M1421: C1401.1, C1402.1, J1401.1 (VTref), J1402.1 (Pin_1), R1404.1, R1405.1, U1401.1 (VCC), U1401.19 (VCC), U1401.22 (VCC), U1401.4 (VCC), U1402.5 (VCC), U1403.5 (VCC), U1404.5 (VCC)
- new net DEV_M1421_NRST: R1404.2, U1404.2
- new net DEV_M1421_SEL: R1401.1, U1402.6 (IN2)
- new net DEV_M1421_SYNC: R1403.1, U1403.2
- new net DEV_M1421_TX: U1402.3 (IN0)
- new net GND: C1401.2, C1402.2, D1401.1 (K), D1402.1 (K), D1403.2 (A2), J1401.3 (GND), J1401.5 (GND), J1401.9 (GNDDetect), J1402.6 (Pin_6), J1403.2 (Ext), R1401.2, R1402.2, R1403.2, U1401.18 (GND), U1401.23 (GND), U1401.25 (GND), U1401.27 (GND), U1401.34 (GND), U1401.36 (GND), U1401.6 (GND), U1401.MP, U1402.2 (GND), U1403.3 (GND), U1404.3 (GND), U1405.1 (GND), U1405.3 (GND), U1405.5 (GND)
- new net LED_SD26_A: D1401.2 (A), R1406.2
- new net LED_SD27_A: D1402.2 (A), R1407.2
- new net M1421_CSCK: TP1410.1, U1401.31 (COPRO_SPI_CLK)
- new net M1421_CSMI: TP1408.1, U1401.29 (COPRO_SPI_MISO)
- new net M1421_CSMO: TP1409.1, U1401.30 (COPRO_SPI_MOSI)
- new net M1421_LBSY: TP1412.1, U1401.33 (LR_BUSY)
- new net M1421_LD08: TP1406.1, U1401.5 (LR_DIO8)
- new net M1421_LD09: TP1405.1, U1401.3 (LR_DIO9)
- new net M1421_LD11: TP1404.1, U1401.2 (LR_DIO11)
- new net M1421_LRCS: TP1411.1, U1401.32 (~{LR_CS})
- new net M1421_LRST: TP1407.1, U1401.7 (~{LR_RESET})
- new net M1421_NRST: J1401.10 (~{RESET}), J1402.5 (Pin_5), R1405.2, U1401.17 (~{SUBG_RESET}), U1404.4
- new net M1421_RF_1090: R1408.1, U1401.26 (LR_RF_LF), U1405.4 (P2)
- new net M1421_RF_978: R1408.2, U1401.24 (SUBG_RF), U1405.6 (P1)
- new net M1421_SD23: TP1401.1, U1401.12 (SUBG_DIO23)
- new net M1421_SD24: TP1402.1, U1401.13 (SUBG_DIO24)
- new net M1421_SD25: TP1403.1, U1401.14 (SUBG_DIO25)
- new net M1421_SD26: R1406.1, U1401.15 (SUBG_DIO26)
- new net M1421_SD27: R1407.1, U1401.16 (SUBG_DIO27)
- new net M1421_SURX: J1402.2 (Pin_2), U1401.20 (SUBG_UART_RX), U1402.4 (Y)
- new net M1421_SUTX: J1402.3 (Pin_3), U1401.21 (SUBG_UART_TX)
- new net M1421_SYNC: J1402.4 (Pin_4), R1402.1, U1401.28 (SYNC), U1403.4
- new net M1421_TCKC: J1401.4 (SWCLK/TCK), U1401.9 (JTAG_TCKC)
- new net M1421_TDI: J1401.8 (NC/TDI), U1401.11 (JTAG_TDI)
- new net M1421_TDO: J1401.6 (SWO/TDO), U1401.10 (JTAG_TDO)
- new net M1421_TMSC: J1401.2 (SWDIO/TMS), U1401.8 (JTAG_TMSC)
- new net P4_M1421_SYNC: U1403.1
- new net P4_M1421_TX: U1402.1 (IN1)
- new net RF_ADSB_ANT: D1403.1 (A1), J1403.1 (In), U1405.2 (SUM)
- no-connect marks 0 -> 3
Other:
- note added: "FIT OPTIONS: (a) solder U1401 m1421, or (b) leave U1401 off and plug the ADSBee 1421 Dev Kit into J1402 with its JST-GH-to-DuPont harness (Dev Kit uses its own U.FL antenna). SYNC (pad 28) is an INPUT: high at reset = ROM bootloader, high at run time = sleep. M1421_NRST: TCA6408A bit 7 drives it open-drain style (output-low = reset, input = release), U1404 for the Dev-port RP2040, J1401 pin 10 fo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"

Commit message: Release v0.18.0: power switch, always-on VBACKUP, hand-solder footprints, PCBWay notes
Co-Authored-By: Claude Opus 5.5 <noreply@anthropic.com>
Parts:
- C1401, C1402: footprint Capacitor_SMD:C_0402_1005Metric -> Capacitor_SMD:C_0805_2012Metric_Pad1.18x1.45mm_HandSolder
- D1401, D1402: footprint LED_SMD:LED_0603_1608Metric -> LED_SMD:LED_0805_2012Metric_Pad1.15x1.40mm_HandSolder
- R1401, R1402, R1403, R1404, R1405, R1406, R1407, R1408: footprint Resistor_SMD:R_0402_1005Metric -> Resistor_SMD:R_0805_2012Metric_Pad1.20x1.40mm_HandSolder
- TP1401, TP1402, TP1403, TP1404, TP1405, TP1406, TP1407, TP1408, TP1409, TP1410, TP1411, TP1412: footprint TestPoint:TestPoint_Pad_D1.0mm -> TestPoint:TestPoint_Pad_D1.5mm

Commit message: Release v0.19.0: hand-solder footprints (m1421, QFNs, SOT-23, SO-8), Rev 1 hand assembly
Co-Authored-By: Claude Opus 5.5 <noreply@anthropic.com>
Parts:
- U1401: footprint ADSB_Test:PantsForBirds_ADSBee_m1421_Module -> ADSB_Test:PantsForBirds_ADSBee_m1421_Module_HandSolder
- U1402: footprint Package_TO_SOT_SMD:SOT-363_SC-70-6 -> Package_TO_SOT_SMD:SOT-23-6_Handsoldering
- U1403, U1404: footprint Package_TO_SOT_SMD:SOT-353_SC-70-5 -> Package_TO_SOT_SMD:SOT-23-5_HandSoldering

Commit message: Release v0.20.0: RF can for m1421, P4+C5 module option (WT01P4C5-S1)
Co-Authored-By: Claude Opus 5.5 <noreply@anthropic.com>
Parts:
- added SH1401: RF can frame (DNP), RF_Shielding:Laird_Technologies_BMI-S-203-F_26.21x26.21mm, symbol Mechanical:Housing_Pad
Connections:
- net GND: now also SH1401.1 (PAD)

Commit message: Release v0.22.0: all ADSB_Test schematic sheets generated (ERC clean)
Co-Authored-By: Claude Opus 5.5 <noreply@anthropic.com>
Parts:
- added R1409: 100k, Resistor_SMD:R_0805_2012Metric_Pad1.20x1.40mm_HandSolder, symbol Device:R
- U1402: value 74LVC1G97 (2:1 mux) -> 74LVC1G97 (AND); Function C(6)=0: Y=B(1)=P4 TX; C(6)=1: Y=A(3)=Dev TX -> B(1)=GND: Y = A(3) AND C(6) = Dev TX AND P4 TX (UART idle h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
Connections:
- net 3V3_M1421: now also R1401.1, R1409.1
- net DEV_M1421_TX: now also R1401.2
- net GND: now also U1402.1 (IN1); no longer R1401.2
- net P4_M1421_TX: now also U1402.6 (IN2), R1409.2; no longer U1402.1 (IN1)
- removed net DEV_M1421_SEL: R1401.1, U1402.6 (IN2)
