File: boards/adsb-test/hardware/kicad/rtc.kicad_sch (KiCad schematic)
At the start: 5 parts, among them U701 DS3231M

Commit message: Release v0.24.0: OSPTEK ESP32-P4C5 Core module replaces WT01P4C5-S1
Co-Authored-By: Claude Opus 5.5 <noreply@anthropic.com>
Parts:
- C701, C702: now not fitted
- U701: DNP (none) -> Optional: fit for +/-5 ppm time keeping; now not fitted
Other:
- note added: "RTC: DS3231M (+/-5 ppm, MEMS resonator, no crystal) at I2C 0x68. VCC from 3V3 when on; VBAT from VBACKUP (always-on 3.0 V LDO, optional CR1220) when off. INT/SQW (open drain) -> P4 GPIO13 (LP GPIO: alarm wake-up from deep sleep). OPTIONAL (DNP): the OSPTEK module has RTC_VBAT on VBACKUP, so the P4 RTC keeps time. Fit U701/C701/C702 for a +/-5 ppm clock (Q27). R701 stays fitted (RTC_INT pull-up)."
- note removed: "RTC: DS3231M (+/-5 ppm, MEMS resonator, no crystal) at I2C 0x68. VCC from 3V3 when on; VBAT from VBACKUP (always-on 3.0 V LDO, optional CR1220) when off. INT/SQW (open drain) -> P4 GPIO6 (LP GPIO: alarm wake-up from deep sleep). Replaces the P4's own RTC backup: the WT01P4C5-S1 has no VBAT pin (Q27)."
