File: boards/adsb-test/hardware/kicad/ADSB_Test.kicad_pcb (KiCad board)
At the start: 4 copper layers, 180.9 x 116 mm, 499 parts, among them J1001 Dev USB-C, J1101 USB-A (SDR hub), J1201 SMA GNSS (active antenna), J1301 LCD FPC 30p 0.5mm, J1302 Touch FPC 6p 0.5mm, J1401 m1421 JTAG (J-Link), J1402 ADSBee 1421 Dev Kit, J1403 SMA 1090/978, J1501 microSD (push-pull, detect), J1601 Kingst LA5016 (2x20 keyed), J1801 RP2040 GPIO (pins DNP), J301 2S Li-ion pack (BAT+, GND, NT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, J601 U.FL Wi-Fi (from module IPEX), J602 RP-SMA Wi-Fi 2.4/5 GHz, J801 HR911105A, J901 User USB-C (PD sink + UART), Q1501 AO3401A, Q1701 MMBT3904, Q1702 MMBT3904, Q1703 MMBT3904, Q1704 MMBT3904, Q201 FDS9435A, SW1801 BOOTSEL (programmer), SW401 POWER (slide), SW601 BOOT, SW602 RESET, SW603 SLEEP/WAKE, U1001 USBLC6-2SC6, U1002 AP2112K-3.3, U1003 USB2514B, U1101 TPS259621DDA, U1102 USBLC6-2SC6, U1201 MAX-M10S, U1301 AP3012KTR-E1, U1302 AP2112K-1.8, U1303 AP3032KTR-G1, U1401 ADSBee m1421, U1402 74LVC1G97 (AND), U1403 74LVC1G32, U1404 74LVC1G07, U1405 SCN-2-11+, U1501 TCA6408APW, U1701 FT2232HL, U1702 93LC56B, U1703 74LVC1G07, U1704 74LVC1G125, U1705 74LVC1G07, U1706 74LVC1G125, U1801 RP2040, U1802 W25Q16JVSS, U1803 74LVC1G125, U1804 74LVC1G125, U1805 74LVC1G125, U1806 74LVC1G125, U201 STUSB4500QTR, U301 BQ25798, U302 MCP1703 3.0V (2 uA Iq), U411 TPS62933, U421 TPS62933, U430 TPS22917, U431 TPS22917, U432 TPS22917, U433 TPS22917, U501 PAC1954 (PM1), U502 PAC1954 (PM2), U503 PAC1954 (PM3), U601 ESP32-P4C5 Core (OSPTEK), U701 DS3231M, U801 LAN8720A, U901 CP2102N-A02-GQFN24, U902 USBLC6-2SC6, Y1001 24MHz, Y1701 12MHz, Y1801 12MHz, Y601 32.768kHz, Y801 25MHz

Commit message: ADSB_Test: Ethernet pairs named _P/_N, net classes restored in the project
- ETH_TXP/TXN/RXP/RXN -> ETH_TX_P/_N, ETH_RX_P/_N; HUB_DN2_M -> HUB_DN2_N.
- gen_pcb.py: pcbnew SaveBoard rewrote ADSB_Test.kicad_pro with empty
  net_settings, so every impedance class had been lost since the PCB start.
  Net settings are now kept across the save; 29 nets back in their classes.

Co-Authored-By: Claude Opus 5.5 <noreply@anthropic.com>
Connections:
- net /Dev USB Hub/HUB_DN2_M renamed /Dev USB Hub/HUB_DN2_N
- net /Ethernet/ETH_RXN renamed /Ethernet/ETH_RX_N
- net /Ethernet/ETH_RXP renamed /Ethernet/ETH_RX_P
- net /Ethernet/ETH_TXN renamed /Ethernet/ETH_TX_N
- net /Ethernet/ETH_TXP renamed /Ethernet/ETH_TX_P

Commit message: ADSB_Test: RP2040 SWD header, monitors and touch put to sleep in bsp_sleep()
- J1802 1x3 SWD header (SWCLK, GND, SWDIO, Pico order) on the Dev
  programmer page; BOM line.
- bsp_sleep(): PAC1954s to sleep mode (5 uA each), GT911 sleep command
  with INT held low; bsp_init() wakes the monitors after a button wake-up.

Co-Authored-By: Claude Opus 5.5 <noreply@anthropic.com>
Parts:
- added J1802: RP2040 SWD, Connector_PinHeader_2.54mm:PinHeader_1x03_P2.54mm_Vertical, B.Cu at (317.9, 214.5)
- moved R1809 63.1 mm to (297.8, 223.9)
- moved U1804 62.4 mm to (298.3, 235.4)
- moved U1805 7.01 mm to (304.6, 235.4)
- moved U1806 7.01 mm to (310.9, 235.4)
- moved Y1801 7.01 mm to (319.5, 235.6)
- moved U1801 6.07 mm to (338.9, 227.4)
- moved TP1801 6.07 mm to (323.4, 224.2)
- moved TP1802 6.07 mm to (327.5, 224.2)
- moved TP1803 6.07 mm to (331.5, 224.2)
- moved R1810 6.07 mm to (303.0, 223.9)
- moved R1811 6.07 mm to (308.3, 223.9)
- moved R1812 6.07 mm to (313.5, 223.9)
- moved R1813 6.07 mm to (318.8, 223.9)
- moved U1803 6.07 mm to (358.2, 224.8)
- moved U1802 6.07 mm to (349.6, 225.9)
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Other:
- board text added: "[Dev m1421 Programmer] 40 parts"
- board text removed: "[Dev m1421 Programmer] 39 parts"

Commit message: ADSB_Test PCB: panel-cable slots from the Waveshare board measurements
LCD slot 22 x 3 mm (74-96 mm across, 42.6-45.6 mm up from the panel's
bottom edge), touch slot 8 x 3 mm (34-42 mm, 49.6-52.6 mm), front view.
Sockets 7 mm inside; module moved between the sockets. Floorplan and docs.

Co-Authored-By: Claude Opus 5.5 <noreply@anthropic.com>
Parts:
- moved J1302 21.5 mm to (146.0, 149.0)
- moved J1301 16.7 mm to (193.0, 156.0)
- moved U601 9.90 mm to (166.1, 146.0)
Other:
- outline, holes or cut-outs redrawn
- board text added: "ADSB_Test Rev A - ALL COMPONENTS ON THE BOTTOM SIDE (panel bonded to the top). Dwgs.User rectangle = panel outline. Slots = panel FPC pass-throughs (from the Waveshare board)."
- board text removed: "ADSB_Test Rev A - ALL COMPONENTS ON THE BOTTOM SIDE (panel bonded to the top). Dwgs.User rectangle = panel outline. Slots = panel FPC pass-throughs (check against the real panel)."
