File: boards/adsb-test/hardware/kicad/dev_prog.kicad_sch (KiCad schematic)
At the start: 41 parts, among them J1801 RP2040 GPIO (pins DNP), SW1801 BOOTSEL (programmer), U1801 RP2040, U1802 W25Q16JVSS, U1803 74LVC1G125, U1804 74LVC1G125, U1805 74LVC1G125, U1806 74LVC1G125, Y1801 12MHz

Commit message: ADSB_Test: RP2040 SWD header, monitors and touch put to sleep in bsp_sleep()
- J1802 1x3 SWD header (SWCLK, GND, SWDIO, Pico order) on the Dev
  programmer page; BOM line.
- bsp_sleep(): PAC1954s to sleep mode (5 uA each), GT911 sleep command
  with INT held low; bsp_init() wakes the monitors after a button wake-up.

Co-Authored-By: Claude Opus 5.5 <noreply@anthropic.com>
Parts:
- added J1802: RP2040 SWD, Connector_PinHeader_2.54mm:PinHeader_1x03_P2.54mm_Vertical, symbol Connector_Generic:Conn_01x03
Connections:
- net GND: now also J1802.2 (Pin_2)
- net RP_SWCLK: now also J1802.1 (Pin_1)
- net RP_SWDIO: now also J1802.3 (Pin_3)
