File: boards/adsb-test/hardware/kicad/ethernet.kicad_sch (KiCad schematic)
At the start: 32 parts, among them J801 HR911105A, U801 LAN8720A, Y801 25MHz

Commit message: ADSB_Test: Ethernet pairs named _P/_N, net classes restored in the project
- ETH_TXP/TXN/RXP/RXN -> ETH_TX_P/_N, ETH_RX_P/_N; HUB_DN2_M -> HUB_DN2_N.
- gen_pcb.py: pcbnew SaveBoard rewrote ADSB_Test.kicad_pro with empty
  net_settings, so every impedance class had been lost since the PCB start.
  Net settings are now kept across the save; 29 nets back in their classes.

Co-Authored-By: Claude Opus 5.5 <noreply@anthropic.com>
Connections:
- net ETH_RXN renamed ETH_RX_N
- net ETH_RXP renamed ETH_RX_P
- net ETH_TXN renamed ETH_TX_N
- net ETH_TXP renamed ETH_TX_P
